Commit message: created model of the human hand

File: sr_antropomorphic/urdf/human_hand.urdf (robot description, URDF)
Before this commit: robot visual, 9 links, 8 joints
Links:
- added link rh_ffdistalphalanx
- added link rh_ffmedialphalanx
- added link rh_ffmetacarpal
- added link rh_ffmpc1
- added link rh_ffmpc2
- added link rh_ffproximalphalanx
- added link rh_fftip
- added link rh_lfcmc
- added link rh_lfdistalphalanx
- added link rh_lfmedialphalanx
- added link rh_lfmetacarpal
- added link rh_lfmpc1
- added link rh_lfmpc2
- added link rh_lfproximalphalanx
- added link rh_lftip
- added link rh_mfdistalphalanx
- added link rh_mfmedialphalanx
- added link rh_mfmetacarpal
- added link rh_mfmpc1
- added link rh_mfmpc2
- added link rh_mfproximalphalanx
- added link rh_mftip
- added link rh_rfcmc
- added link rh_rfdistalphalanx
- added link rh_rfmedialphalanx
- added link rh_rfmetacarpal
- added link rh_rfmpc1
- added link rh_rfmpc2
- added link rh_rfproximalphalanx
- added link rh_rftip
- added link world
Joints:
- added joint ffdistalphalanx_to_fftip: type fixed, parent rh_ffdistalphalanx, child rh_fftip, origin xyz=0.0 0.097 0.0 rpy=0.0 0.0 0.0
- added joint ffmedialphalanx_to_ffdistalphalanx: type revolute, parent rh_ffmedialphalanx, child rh_ffdistalphalanx, origin xyz=0.0 0.143 0.0 rpy=0.0 0.0 0.0, axis 0 0 1, limit lower=0.0 upper=1.570796327 effort=1000.0 velocity=0.5
- added joint ffmetacarpal_to_ffmpc1: type revolute, parent rh_ffproximalphalanx, child rh_ffmpc1, origin xyz=0.0 0.0 0.0 rpy=0.0 0.0 0.0, axis 1 0 0, limit lower=-0.2617993878 upper=0.7330382858 effort=1000.0 velocity=0.5
- added joint ffmetacarpal_to_ffproximalphalanx: type fixed, parent rh_ffmetacarpal, child rh_ffproximalphalanx, origin xyz=0.0 0.3779 0.0 rpy=-0.2618 0.0 0.0
- added joint ffmpc1_to_ffmpc2: type revolute, parent rh_ffmpc1, child rh_ffmpc2, origin xyz=0.0 0.0 0.0 rpy=0.0 0.0 0.0, axis 0 0 1, limit lower=0.0 upper=1.570796327 effort=1000.0 velocity=0.5
- added joint ffmpc2_to_ffmedialphalanx: type revolute, parent rh_ffmpc2, child rh_ffmedialphalanx, origin xyz=0.0 0.2649 0.0 rpy=0.0 0.0 0.0, axis 0 0 1, limit lower=0.0 upper=1.745329252 effort=1000.0 velocity=0.5
- added joint lfdistalphalanx_to_rftip: type fixed, parent rh_lfdistalphalanx, child rh_lftip, origin xyz=0.0 0.093 0.0 rpy=0.0 0.0 0.0
- added joint lfmedialphalanx_to_lfdistalphalanx: type revolute, parent rh_lfmedialphalanx, child rh_lfdistalphalanx, origin xyz=0.0 0.117 0.0 rpy=0.0 0.0 0.0, axis 0 0 1, limit lower=0.0 upper=1.570796327 effort=1000.0 velocity=0.5
- added joint lfmetacarpal_to_lfmpc1: type revolute, parent rh_lfproximalphalanx, child rh_lfmpc1, origin xyz=0.0 0.0 0.0 rpy=0.0 0.0 0.0, axis 1 0 0, limit lower=-0.6981317008 upper=0.3316125579 effort=1000.0 velocity=0.5
- added joint lfmetacarpal_to_lfproximalphalanx: type fixed, parent rh_lfcmc, child rh_lfproximalphalanx, origin xyz=0.0 0.3049 0.0 rpy=0.1222 0.0 0.0
- added joint lfmpc1_to_lfmpc2: type revolute, parent rh_lfmpc1, child rh_lfmpc2, origin xyz=0.0 0.0 0.0 rpy=0.0 0.0 0.0, axis 0 0 1, limit lower=0.0 upper=1.570796327 effort=1000.0 velocity=0.5
- added joint lfmpc2_to_lfmedialphalanx: type revolute, parent rh_lfmpc2, child rh_lfmedialphalanx, origin xyz=0.0 0.2059 0.0 rpy=0.0 0.0 0.0, axis 0 0 1, limit lower=0.0 upper=1.745329252 effort=1000.0 velocity=0.5
- added joint mfdistalphalanx_to_mftip: type fixed, parent rh_mfdistalphalanx, child rh_mftip, origin xyz=0.0 0.108 0.0 rpy=0.0 0.0 0.0
- added joint mfmedialphalanx_to_mfdistalphalanx: type revolute, parent rh_mfmedialphalanx, child rh_mfdistalphalanx, origin xyz=0.0 0.17 0.0 rpy=0.0 0.0 0.0, axis 0 0 1, limit lower=0.0 upper=1.570796327 effort=1000.0 velocity=0.5
- added joint mfmetacarpal_to_mfmpc1: type revolute, parent rh_mfproximalphalanx, child rh_mfmpc1, origin xyz=0.0 0.0 0.0 rpy=0.0 0.0 0.0, axis 1 0 0, limit lower=-0.1396263402 upper=0.6108652382 effort=1000.0 velocity=0.5
- added joint mfmetacarpal_to_mfproximalphalanx: type fixed, parent rh_mfmetacarpal, child rh_mfproximalphalanx, origin xyz=0.0 0.377 0.0 rpy=-0.1047 0.0 0.0
- added joint mfmpc1_to_mfmpc2: type revolute, parent rh_mfmpc1, child rh_mfmpc2, origin xyz=0.0 0.0 0.0 rpy=0.0 0.0 0.0, axis 0 0 1, limit lower=0.0 upper=1.570796327 effort=1000.0 velocity=0.5
- added joint mfmpc2_to_mfmedialphalanx: type revolute, parent rh_mfmpc2, child rh_mfmedialphalanx, origin xyz=0.0 0.2773 0.0 rpy=0.0 0.0 0.0, axis 0 0 1, limit lower=0.0 upper=1.745329252 effort=1000.0 velocity=0.5
- added joint palm_to_ffmetacarpal: type fixed, parent rh_palm, child rh_ffmetacarpal, origin xyz=0.0 0.073 0.0541 rpy=0.1438 0.0 0.0
- added joint palm_to_lfmetacarpal: type fixed, parent rh_palm, child rh_lfmetacarpal, origin xyz=0.0 0.073 -0.0958 rpy=-0.2427 0.0 0.0
- added joint palm_to_mfmetacarpal: type fixed, parent rh_palm, child rh_mfmetacarpal, origin xyz=0.0 0.073 0.0 rpy=0.0 0.0 0.0
- added joint palm_to_rfmetacarpal: type fixed, parent rh_palm, child rh_rfmetacarpal, origin xyz=0.0 0.073 -0.0554 rpy=-0.0981 0.0 0.0
- added joint rfdistalphalanx_to_rftip: type fixed, parent rh_rfdistalphalanx, child rh_rftip, origin xyz=0.0 0.107 0.0 rpy=0.0 0.0 0.0
- added joint rfmedialphalanx_to_rfdistalphalanx: type revolute, parent rh_rfmedialphalanx, child rh_rfdistalphalanx, origin xyz=0.0 0.165 0.0 rpy=0.0 0.0 0.0, axis 0 0 1, limit lower=0.0 upper=1.570796327 effort=1000.0 velocity=0.5
- added joint rfmetacarpal_to_lfcmc: type revolute, parent rh_lfmetacarpal, child rh_lfcmc, origin xyz=0.0 0.0 0.0 rpy=0.0 0.0 0.0, axis 0 1 0, limit lower=0.0 upper=0.5235987756 effort=1000.0 velocity=0.5
- added joint rfmetacarpal_to_rfcmc: type revolute, parent rh_rfmetacarpal, child rh_rfcmc, origin xyz=0.0 0.0 0.0 rpy=0.0 0.0 0.0, axis 0 1 0, limit lower=0.0 upper=0.2617993878 effort=1000.0 velocity=0.5
- added joint rfmetacarpal_to_rfmpc1: type revolute, parent rh_rfproximalphalanx, child rh_rfmpc1, origin xyz=0.0 0.0 0.0 rpy=0.0 0.0 0.0, axis 1 0 0, limit lower=-0.3490658504 upper=0.2443460953 effort=1000.0 velocity=0.5
- added joint rfmetacarpal_to_rfproximalphalanx: type fixed, parent rh_rfcmc, child rh_rfproximalphalanx, origin xyz=0.0 0.3376 0.0 rpy=0.0 0.0 0.0
- added joint rfmpc1_to_rfmpc2: type revolute, parent rh_rfmpc1, child rh_rfmpc2, origin xyz=0.0 0.0 0.0 rpy=0.0 0.0 0.0, axis 0 0 1, limit lower=0.0 upper=1.570796327 effort=1000.0 velocity=0.5
- added joint rfmpc2_to_rfmedialphalanx: type revolute, parent rh_rfmpc2, child rh_rfmedialphalanx, origin xyz=0.0 0.2591 0.0 rpy=0.0 0.0 0.0, axis 0 0 1, limit lower=0.0 upper=1.745329252 effort=1000.0 velocity=0.5
- added joint world_to_palm: type fixed, parent world, child rh_palm, origin xyz=0 0 0 rpy=0.0 -1.57079632679 3.14159265359
- joint thcmc1_to_thcmc2: axis (none) -> 0 0 1; origin xyz=0.0 0.0 0.0 rpy=0.0 0.0 1.57079632679 -> xyz=0.0 0.0 0.0 rpy=0.0 0.0 0.0
- joint thcmc2_to_thproximalphalanx: axis (none) -> 0 0 1; origin xyz=0.251 0.0 0.0 rpy=0.0 0.0 0.0 -> xyz=0.0 0.251 0.0 rpy=0.0 0.0 0.0
- joint thmpc_to_thmedialphalanx: axis (none) -> 0 0 1; origin xyz=0.196 0.0 0.0 rpy=0.0 0.0 0.0 -> xyz=0.0 0.196 0.0 rpy=0.0 0.0 0.0
- joint thproximalphalanx_to_thmpc: axis (none) -> 1 0 0

Commit message: add ext

File: sr_antropomorphic/urdf/human_hand.urdf (robot description, URDF)
Before this commit: robot visual, 40 links, 39 joints
Links:
- removed link rh_ffmpc1
- removed link rh_ffmpc2
- removed link rh_lfmpc1
- removed link rh_lfmpc2
- removed link rh_mfmpc1
- removed link rh_mfmpc2
- removed link rh_rfmpc1
- removed link rh_rfmpc2
- removed link rh_thcmc1
- removed link rh_thcmc2
- removed link rh_thmpc
- added link rh_ffmpcadd
- added link rh_ffmpcext
- added link rh_lfmpcadd
- added link rh_lfmpcext
- added link rh_mfmpcadd
- added link rh_mfmpcext
- added link rh_rfmpcadd
- added link rh_rfmpcext
- added link rh_thcmcadd
- added link rh_thcmcext
- added link rh_thmpext
Joints:
- removed joint ffmetacarpal_to_ffmpc1
- removed joint ffmpc1_to_ffmpc2
- removed joint ffmpc2_to_ffmedialphalanx
- removed joint lfmetacarpal_to_lfmpc1
- removed joint lfmpc1_to_lfmpc2
- removed joint lfmpc2_to_lfmedialphalanx
- removed joint mfmetacarpal_to_mfmpc1
- removed joint mfmpc1_to_mfmpc2
- removed joint mfmpc2_to_mfmedialphalanx
- removed joint rfmetacarpal_to_rfmpc1
- removed joint rfmpc1_to_rfmpc2
- removed joint rfmpc2_to_rfmedialphalanx
- removed joint thcmc1_to_thcmc2
- removed joint thcmc2_to_thproximalphalanx
- removed joint thmetacarpal_to_thcmc1
- added joint ffmetacarpal_to_ffmpcadd: type revolute, parent rh_ffproximalphalanx, child rh_ffmpcadd, origin xyz=0.0 0.0 0.0 rpy=0.0 0.0 0.0, axis 1 0 0, limit lower=-0.2617993878 upper=0.7330382858 effort=1000.0 velocity=0.5
- added joint ffmpcadd_to_ffmpcext: type revolute, parent rh_ffmpcadd, child rh_ffmpcext, origin xyz=0.0 0.0 0.0 rpy=0.0 0.0 0.0, axis 0 0 1, limit lower=0.0 upper=1.570796327 effort=1000.0 velocity=0.5
- added joint ffmpcext_to_ffmedialphalanx: type revolute, parent rh_ffmpcext, child rh_ffmedialphalanx, origin xyz=0.0 0.2649 0.0 rpy=0.0 0.0 0.0, axis 0 0 1, limit lower=0.0 upper=1.745329252 effort=1000.0 velocity=0.5
- added joint lfmetacarpal_to_lfmpcadd: type revolute, parent rh_lfproximalphalanx, child rh_lfmpcadd, origin xyz=0.0 0.0 0.0 rpy=0.0 0.0 0.0, axis 1 0 0, limit lower=-0.6981317008 upper=0.3316125579 effort=1000.0 velocity=0.5
- added joint lfmpcadd_to_lfmpcext: type revolute, parent rh_lfmpcadd, child rh_lfmpcext, origin xyz=0.0 0.0 0.0 rpy=0.0 0.0 0.0, axis 0 0 1, limit lower=0.0 upper=1.570796327 effort=1000.0 velocity=0.5
- added joint lfmpcext_to_lfmedialphalanx: type revolute, parent rh_lfmpcext, child rh_lfmedialphalanx, origin xyz=0.0 0.2059 0.0 rpy=0.0 0.0 0.0, axis 0 0 1, limit lower=0.0 upper=1.745329252 effort=1000.0 velocity=0.5
- added joint mfmetacarpal_to_mfmpcadd: type revolute, parent rh_mfproximalphalanx, child rh_mfmpcadd, origin xyz=0.0 0.0 0.0 rpy=0.0 0.0 0.0, axis 1 0 0, limit lower=-0.1396263402 upper=0.6108652382 effort=1000.0 velocity=0.5
- added joint mfmpcadd_to_mfmpcext: type revolute, parent rh_mfmpcadd, child rh_mfmpcext, origin xyz=0.0 0.0 0.0 rpy=0.0 0.0 0.0, axis 0 0 1, limit lower=0.0 upper=1.570796327 effort=1000.0 velocity=0.5
- added joint mfmpcext_to_mfmedialphalanx: type revolute, parent rh_mfmpcext, child rh_mfmedialphalanx, origin xyz=0.0 0.2773 0.0 rpy=0.0 0.0 0.0, axis 0 0 1, limit lower=0.0 upper=1.745329252 effort=1000.0 velocity=0.5
- added joint rfmetacarpal_to_rfmpcadd: type revolute, parent rh_rfproximalphalanx, child rh_rfmpcadd, origin xyz=0.0 0.0 0.0 rpy=0.0 0.0 0.0, axis 1 0 0, limit lower=-0.3490658504 upper=0.2443460953 effort=1000.0 velocity=0.5
- added joint rfmpcadd_to_rfmpcext: type revolute, parent rh_rfmpcadd, child rh_rfmpcext, origin xyz=0.0 0.0 0.0 rpy=0.0 0.0 0.0, axis 0 0 1, limit lower=0.0 upper=1.570796327 effort=1000.0 velocity=0.5
- added joint rfmpcext_to_rfmedialphalanx: type revolute, parent rh_rfmpcext, child rh_rfmedialphalanx, origin xyz=0.0 0.2591 0.0 rpy=0.0 0.0 0.0, axis 0 0 1, limit lower=0.0 upper=1.745329252 effort=1000.0 velocity=0.5
- added joint thcmcadd_to_thcmcext: type revolute, parent rh_thcmcadd, child rh_thcmcext, origin xyz=0.0 0.0 0.0 rpy=0.0 0.0 0.0, axis 1 0 0, limit lower=-0.436332313 upper=0.6108652382 effort=1000.0 velocity=0.5
- added joint thcmcext_to_thproximalphalanx: type revolute, parent rh_thcmcext, child rh_thproximalphalanx, origin xyz=0.0 0.251 0.0 rpy=0.0 0.0 0.0, axis 0 0 1, limit lower=-0.5235987756 upper=1.047197551 effort=1000.0 velocity=0.5
- added joint thmetacarpal_to_thcmcadd: type revolute, parent rh_thmetacarpal, child rh_thcmcadd, origin xyz=0.0 0.0 0.0 rpy=0.0 0.0 0.0, axis 0 0 1, limit lower=-0.5235987756 upper=1.047197551 effort=1000.0 velocity=0.5
- joint thmpc_to_thmedialphalanx: parent rh_thmpc -> rh_thmpext
- joint thproximalphalanx_to_thmpc: child rh_thmpc -> rh_thmpext
